File: KiCad/CERS.kicad_pcb (KiCad board)
At the start: 2 copper layers, 60 x 90 mm, 17 parts, among them J1 NFC, J2 PWR, J3 OLED, SW1 IN/OUT, SW2 CONF, U1 ESP32-DEVKITC

Commit message: Fix R1 value.
Parts:
- R1: value 120 -> 1k
Changed lines of the file:
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@@
       (effects (font (size 1 1) (thickness 0.15)))
     )
-    (fp_text value 120 (at 5.08 2.37 90) (layer F.Fab)
+    (fp_text value 1k (at 5.08 2.37 90) (layer F.Fab)
       (effects (font (size 1 1) (thickness 0.15)))
     )

Commit message: Update KiCad files rev. 1.1
Parts:
- added R2: 1k, Resistor_THT:R_Axial_DIN0207_L6.3mm_D2.5mm_P10.16mm_Horizontal, F.Cu at (65.0, 54.0)
- D1: value STAT -> GL8ED48; footprint LED_THT:LED_D2.0mm_W4.8mm_H2.5mm_FlatTop -> LED_THT:LED_D3.0mm-3
- moved D1 3.65 mm to (41.5, 28.5), turned to 0 degrees
Connections:
- D1 pad 1: GND -> Net-(D1-Pad1)
- D1 pad 2: Net-(D1-Pad2) -> GND
- R1 pad 2: Net-(D1-Pad2) -> Net-(D1-Pad1)
Routing:
- net Net-(D1-Pad3): track 0.00 -> 28.5 mm
- net Net-(D1-Pad1): track 0.00 -> 28.0 mm
- net Net-(D1-Pad2): track 23.9 -> 0.00 mm
- net GND: track 149.8 -> 159.2 mm
- net Net-(R2-Pad1): track 0.00 -> 7.19 mm
